Commit message: added camera

File: src/ros2_so_arm100/so_arm101_description/control/so_arm101.ros2_control.xacro (robot description, xacro)
@@ -57,5 +57,7 @@
         <param name="initial_position">0.0</param>
         <command_interface name="position" />
-        <state_interface name="position" />
+        <state_interface name="position">
+          <param name="initial_value">1.5708</param>
+        </state_interface>
         <state_interface name="velocity" />
       </joint>

File: src/ros2_so_arm100/so_arm101_description/urdf/so_arm101_macro.xacro (robot description, xacro)
@@ -567,5 +567,4 @@
     </transmission>
     <!-- Joint from upper_arm to lower_arm -->
-    <!-- Note: 5-degree calibration offset applied to joint limits -->
     <joint name="${prefix}elbow_flex_joint" type="revolute">
       <origin
@@ -576,5 +575,5 @@
       <child link="${prefix}lower_arm_link" />
       <axis xyz="0 0 1" />
-      <limit effort="10" velocity="10" lower="-1.69" upper="1.54" />
+      <limit effort="10" velocity="10" lower="-1.69" upper="1.69" />
     </joint>
     <transmission name="${prefix}elbow_flex_trans">
@@ -596,10 +595,10 @@
       <origin
         xyz="-0.1349 0.0052 3.62355e-17"
-        rpy="-1.41553e-15 4.91611e-15 -1.57"
+        rpy="4.02456e-15 8.67362e-16 -1.5708"
       />
       <parent link="${prefix}lower_arm_link" />
       <child link="${prefix}wrist_link" />
       <axis xyz="0 0 1" />
-      <limit effort="10" velocity="10" lower="-1.6" upper="1.6" />
+      <limit effort="10" velocity="10" lower="-1.65806" upper="1.65806" />
     </joint>
     <transmission name="${prefix}wrist_flex_trans">
@@ -619,9 +618,9 @@
     <!-- Joint from wrist to gripper -->
     <joint name="${prefix}wrist_roll_joint" type="revolute">
-      <origin xyz="0.0 -0.0611  0.0181" rpy="-1.57 3.14 0" />
+      <origin xyz="5.55112e-17 -0.0611 0.0181" rpy="1.5708 0.0486795 3.14159" />
       <parent link="${prefix}wrist_link" />
       <child link="${prefix}gripper_link" />
       <axis xyz="0 0 1" />
-      <limit effort="10" velocity="10" lower="-2.3" upper="2.3" />
+      <limit effort="10" velocity="10" lower="-2.74385" upper="2.84121" />
     </joint>
     <transmission name="${prefix}wrist_roll_trans">
@@ -648,9 +647,9 @@
     <!-- Joint from gripper to jaw -->
     <joint name="${prefix}gripper_joint" type="revolute">
-      <origin xyz="0.0202 0.0188 -0.0234" rpy="1.5708 0.18 -1.41553e-15" />
+      <origin xyz="0.0202 0.0188 -0.0234" rpy="1.5708 -5.24284e-08 -1.41553e-15" />
       <parent link="${prefix}gripper_link" />
       <child link="${prefix}jaw_link" />
       <axis xyz="0 0 1" />
-      <limit effort="10" velocity="10" lower="0.0" upper="1.70" />
+      <limit effort="10" velocity="10" lower="-0.174533" upper="1.74533" />
     </joint>
     <transmission name="${prefix}gripper_trans">
