Commit message: early vision tested, corrected camera shape and orientation, changed tracking for png output

File: src/ros2_so_arm100/so_arm_gz/camera/camera.xacro (robot description, xacro)
@@ -4,8 +4,9 @@
     <color rgba="1.0 0.0 0.0 1.0"/>
   </material>
+  <!--ONLY dimensions, weight, and inertia match the values of a orbbec femto bolt camera. Sensor specs are custom-->
   <link name="camera_link">
     <visual>
       <geometry>
-        <box size="0.1 0.1 0.1"/>
+        <box size="0.04026 0.1153 0.06495"/>
       </geometry>
       <material name="red"/>
@@ -13,11 +14,11 @@
     <collision>
       <geometry>
-        <box size="0.1 0.1 0.1"/>
+        <box size="0.04026 0.1153 0.06495"/>
       </geometry>
     </collision>
     <inertial>
-      <mass value="0.05"/>
+      <mass value="0.348"/>
       <origin xyz="0.0 0.0 0.0" rpy="0.0 0.0 0.0"/>
-      <inertia ixx="0.0001" ixy="0.0" ixz="0.0" iyy="0.0001" iyz="0.0" izz="0.0001"/>
+      <inertia ixx="5.08e-4" ixy="0.0" ixz="0.0" iyy="1.69e-4" iyz="0.0" izz="4.33e-4"/>
     </inertial>
   </link>
